Commit message: unified model with taurob

File: taurob_schunk_lwa4d/urdf/lwa4d/lwa4d.urdf.xacro (robot description, xacro)
@@ -1,8 +1,7 @@
-<?xml version="1.0"?>
 <robot xmlns:xacro="http://www.ros.org/wiki/xacro">
   <xacro:property name="safety_offset" value="0.02"/>
-  <xacro:include filename="$(find schunk_description)/urdf/common.xacro" />
-  <xacro:include filename="$(find schunk_description)/urdf/lwa4d/lwa4d.gazebo.xacro"/>
-  <xacro:include filename="$(find schunk_description)/urdf/lwa4d/lwa4d.transmission.xacro"/>
+  <xacro:include filename="$(find taurob_schunk_lwa4d)/urdf/common.xacro" />
+  <xacro:include filename="$(find taurob_schunk_lwa4d)/urdf/lwa4d/lwa4d.gazebo.xacro"/>
+  <xacro:include filename="$(find taurob_schunk_lwa4d)/urdf/lwa4d/lwa4d.transmission.xacro"/>
   <xacro:macro name="axis_config" params="invert">
     <xacro:if value="${invert}">
@@ -11,4 +10,21 @@
     <xacro:unless value="${invert}">
       <axis xyz="0 0 -1" />
+    </xacro:unless>
+  </xacro:macro>
+  <!-- use_factory_setings is a xacro parameter to be used to adapt the urdf according to your hardware setup.
+       use_factory_settings:=true if you have not modified the schunk firmware.
+       use_factory_settings:=false if you have modified the schunk firmware to follow DH parameters (you have inverted the PRL+ motors j1-j5)
+       if you are using custom firmware settings, use schunk_lwa4d_custom
+  -->
+  <xacro:macro name="schunk_lwa4d" params="parent name *origin has_podest use_factory_settings:=false">
+    <xacro:if value="${use_factory_settings}">
+      <xacro:schunk_lwa4d_custom parent="${parent}" name="${name}" has_podest="${has_podest}" invert_j1="false" invert_j2="false" invert_j3="false" invert_j4="false" invert_j5="false" invert_j6="true" invert_j7="true">
+        <xacro:insert_block name="origin" />
+      </xacro:schunk_lwa4d_custom>
+    </xacro:if>
+    <xacro:unless value="${use_factory_settings}">
+      <xacro:schunk_lwa4d_custom parent="${parent}" name="${name}" has_podest="${has_podest}" invert_j1="true" invert_j2="true" invert_j3="true" invert_j4="true" invert_j5="true" invert_j6="true" invert_j7="true">
+        <xacro:insert_block name="origin" />
+      </xacro:schunk_lwa4d_custom>
     </xacro:unless>
   </xacro:macro>
@@ -264,20 +280,3 @@
     </gazebo>
   </xacro:macro>
-  <!-- use_factory_setings is a xacro parameter to be used to adapt the urdf according to your hardware setup.
-       use_factory_settings:=true if you have not modified the schunk firmware.
-       use_factory_settings:=false if you have modified the schunk firmware to follow DH parameters (you have inverted the PRL+ motors j1-j5)
-       if you are using custom firmware settings, use schunk_lwa4d_custom
-  -->
-  <xacro:macro name="schunk_lwa4d" params="parent name *origin has_podest use_factory_settings:=false">
-    <xacro:if value="${use_factory_settings}">
-      <xacro:schunk_lwa4d_custom parent="${parent}" name="${name}" has_podest="${has_podest}" invert_j1="false" invert_j2="false" invert_j3="false" invert_j4="false" invert_j5="false" invert_j6="true" invert_j7="true">
-        <xacro:insert_block name="origin" />
-      </xacro:schunk_lwa4d_custom>
-    </xacro:if>
-    <xacro:unless value="${use_factory_settings}">
-      <xacro:schunk_lwa4d_custom parent="${parent}" name="${name}" has_podest="${has_podest}" invert_j1="true" invert_j2="true" invert_j3="true" invert_j4="true" invert_j5="true" invert_j6="true" invert_j7="true">
-        <xacro:insert_block name="origin" />
-      </xacro:schunk_lwa4d_custom>
-    </xacro:unless>
-  </xacro:macro>
 </robot>

File: taurob_schunk_lwa4d/urdf/schunk_lwa4d_standalone.urdf.xacro (robot description, xacro)
@@ -6,5 +6,5 @@
   <!-- schunk lwa4d -->
   <xacro:include filename="$(find taurob_schunk_lwa4d)/urdf/lwa4d/lwa4d.urdf.xacro" />
-  <!-- Used for fixing robot to Gazebo -->
+ <!-- Used for fixing robot to Gazebo -->
   <link name="world"/>
   <!-- arm -->

Commit message: several fixies, mostly on model

File: taurob_schunk_lwa4d/urdf/lwa4d/lwa4d.urdf.xacro (robot description, xacro)
@@ -17,5 +17,5 @@
        if you are using custom firmware settings, use schunk_lwa4d_custom
   -->
-  <xacro:macro name="schunk_lwa4d" params="parent name *origin has_podest use_factory_settings:=false">
+  <xacro:macro name="schunk_lwa4d" params="parent name *origin has_podest use_factory_settings">
     <xacro:if value="${use_factory_settings}">
       <xacro:schunk_lwa4d_custom parent="${parent}" name="${name}" has_podest="${has_podest}" invert_j1="false" invert_j2="false" invert_j3="false" invert_j4="false" invert_j5="false" invert_j6="true" invert_j7="true">
@@ -45,5 +45,5 @@
         <visual>
           <geometry>
-            <mesh filename="package://schunk_description/meshes/lwa4d/arm_podest_link.stl"/>
+            <mesh filename="package://taurob_schunk_lwa4d/meshes/lwa4d/arm_podest_link.stl"/>
           </geometry>
           <material name="Schunk/LightGrey"/>
@@ -51,5 +51,5 @@
         <collision>
           <geometry>
-            <mesh filename="package://schunk_description/meshes/lwa4d/arm_podest_link.stl"/>
+            <mesh filename="package://taurob_schunk_lwa4d/meshes/lwa4d/arm_podest_link.stl"/>
           </geometry>
         </collision>
@@ -89,11 +89,11 @@
       <visual>
         <geometry>
-          <mesh filename="package://schunk_description/meshes/lwa4d/arm_1_link.stl"/>
-        </geometry>
-        <material name="Schunk/LightGrey"/>
-      </visual>
-      <collision>
-        <geometry>
-          <mesh filename="package://schunk_description/meshes/lwa4d/arm_1_link.stl"/>
+          <mesh filename="package://taurob_schunk_lwa4d/meshes/lwa4d/arm_1_link.stl"/>
+        </geometry>
+        <material name="Schunk/LightGrey"/>
+      </visual>
+      <collision>
+        <geometry>
+          <mesh filename="package://taurob_schunk_lwa4d/meshes/lwa4d/arm_1_link.stl"/>
         </geometry>
       </collision>
@@ -116,5 +116,5 @@
       <visual>
         <geometry>
-          <mesh filename="package://schunk_description/meshes/lwa4d/arm_2_link.stl"/>
+          <mesh filename="package://taurob_schunk_lwa4d/meshes/lwa4d/arm_2_link.stl"/>
         </geometry>
         <material name="Schunk/Black"/>
@@ -122,5 +122,5 @@
       <collision>
         <geometry>
-          <mesh filename="package://schunk_description/meshes/lwa4d/arm_2_link_collision.stl"/>
+          <mesh filename="package://taurob_schunk_lwa4d/meshes/lwa4d/arm_2_link_collision.stl"/>
         </geometry>
       </collision>
@@ -143,11 +143,11 @@
       <visual>
         <geometry>
-          <mesh filename="package://schunk_description/meshes/lwa4d/arm_3_link.stl"/>
-        </geometry>
-        <material name="Schunk/LightGrey"/>
-      </visual>
-      <collision>
-        <geometry>
-          <mesh filename="package://schunk_description/meshes/lwa4d/arm_3_link_collision.stl"/>
+          <mesh filename="package://taurob_schunk_lwa4d/meshes/lwa4d/arm_3_link.stl"/>
+        </geometry>
+        <material name="Schunk/LightGrey"/>
+      </visual>
+      <collision>
+        <geometry>
+          <mesh filename="package://taurob_schunk_lwa4d/meshes/lwa4d/arm_3_link_collision.stl"/>
         </geometry>
       </collision>
@@ -170,5 +170,5 @@
       <visual>
         <geometry>
-          <mesh filename="package://schunk_description/meshes/lwa4d/arm_4_link.stl"/>
+          <mesh filename="package://taurob_schunk_lwa4d/meshes/lwa4d/arm_4_link.stl"/>
         </geometry>
         <material name="Schunk/Black"/>
@@ -176,5 +176,5 @@
       <collision>
         <geometry>
-          <mesh filename="package://schunk_description/meshes/lwa4d/arm_4_link_collision.stl"/>
+          <mesh filename="package://taurob_schunk_lwa4d/meshes/lwa4d/arm_4_link_collision.stl"/>
         </geometry>
       </collision>
@@ -197,11 +197,11 @@
       <visual>
         <geometry>
-          <mesh filename="package://schunk_description/meshes/lwa4d/arm_5_link.stl"/>
-        </geometry>
-        <material name="Schunk/LightGrey"/>
-      </visual>
-      <collision>
-        <geometry>
-          <mesh filename="package://schunk_description/meshes/lwa4d/arm_5_link_collision.stl"/>
+          <mesh filename="package://taurob_schunk_lwa4d/meshes/lwa4d/arm_5_link.stl"/>
+        </geometry>
+        <material name="Schunk/LightGrey"/>
+      </visual>
+      <collision>
+        <geometry>
+          <mesh filename="package://taurob_schunk_lwa4d/meshes/lwa4d/arm_5_link_collision.stl"/>
         </geometry>
       </collision>
@@ -224,5 +224,5 @@
       <visual>
         <geometry>
-          <mesh filename="package://schunk_description/meshes/lwa4d/arm_6_link.stl"/>
+          <mesh filename="package://taurob_schunk_lwa4d/meshes/lwa4d/arm_6_link.stl"/>
         </geometry>
         <material name="Schunk/Black"/>
@@ -230,5 +230,5 @@
       <collision>
         <geometry>
-          <mesh filename="package://schunk_description/meshes/lwa4d/arm_6_link_collision.stl"/>
+          <mesh filename="package://taurob_schunk_lwa4d/meshes/lwa4d/arm_6_link_collision.stl"/>
         </geometry>
       </collision>
@@ -251,11 +251,11 @@
       <visual>
         <geometry>
-          <mesh filename="package://schunk_description/meshes/lwa4d/arm_7_link.stl"/>
-        </geometry>
-        <material name="Schunk/LightGrey"/>
-      </visual>
-      <collision>
-        <geometry>
-          <mesh filename="package://schunk_description/meshes/lwa4d/arm_7_link.stl"/>
+          <mesh filename="package://taurob_schunk_lwa4d/meshes/lwa4d/arm_7_link.stl"/>
+        </geometry>
+        <material name="Schunk/LightGrey"/>
+      </visual>
+      <collision>
+        <geometry>
+          <mesh filename="package://taurob_schunk_lwa4d/meshes/lwa4d/arm_7_link.stl"/>
         </geometry>
       </collision>

File: taurob_schunk_lwa4d/urdf/schunk_lwa4d_standalone.urdf.xacro (robot description, xacro)
@@ -9,6 +9,6 @@
   <link name="world"/>
   <!-- arm -->
-  <xacro:schunk_lwa4d name="arm" parent="world" has_podest="true">
-    <origin xyz="0 0 0.026" rpy="0 0 0" /> <!--slightly above gazebo plane-->
+  <xacro:schunk_lwa4d name="arm" parent="world" has_podest="true" use_factory_settings="true">
+    <origin xyz="0 0 0" rpy="0 0 0" />
   </xacro:schunk_lwa4d>
 </robot>
