Commit message: gripped support updated

File: erl_schunk_pg70/urdf/pg70/pg70.transmission.xacro (robot description, xacro)
@@ -1,5 +1,5 @@
 <?xml version="1.0"?>
 <robot xmlns:xacro="http://www.ros.org/wiki/xacro">
-  <xacro:include filename="$(find taurob_schunk_lwa4d)/urdf/common.xacro" />
+  <xacro:include filename="$(find erl_schunk_pg70)/urdf/common.xacro" />
   <xacro:macro name="schunk_pg70_transmission" params="name">
     <xacro:default_transmission jname="${name}_finger_left"/>

File: erl_schunk_pg70/urdf/pg70/pg70.urdf.xacro (robot description, xacro)
@@ -1,36 +1,8 @@
 <?xml version="1.0"?>
 <robot xmlns:xacro="http://www.ros.org/wiki/xacro">
-  <xacro:include filename="$(find schunk_description)/urdf/common.xacro" />
-  <xacro:include filename="$(find schunk_description)/urdf/pg70/pg70.gazebo.xacro" />
-  <xacro:include filename="$(find schunk_description)/urdf/pg70/pg70.transmission.xacro" />
-  <xacro:macro name="schunk_pg70" params="parent name *origin has_podest">
-    <xacro:if value="${has_podest}">
-      <joint name="${name}_podest_joint" type="fixed">
-        <xacro:insert_block name="origin" />
-        <parent link="${parent}"/>
-        <child link="${name}_podest_link"/>
-      </joint>
-      <link name="${name}_podest_link">
-        <xacro:default_inertial/>
-        <visual>
-          <origin xyz="0 0 0" rpy="0 ${M_PI} 0" />
-          <geometry>
-          <mesh filename="package://schunk_description/meshes/lwa4p/arm_base_link.stl" />
-          </geometry>
-        </visual>
-        <collision>
-          <origin xyz="0 0 0" rpy="0 ${M_PI} 0" />
-          <geometry>
-          <mesh filename="package://schunk_description/meshes/lwa4p/arm_base_link.stl" />
-          </geometry>
-        </collision>
-      </link>
-      <joint name="${name}_palm_joint" type="fixed">
-        <origin xyz="0 0 0.10" rpy="0 0 0" />
-        <parent link="${name}_podest_link"/>
-        <child link="${name}_palm_link"/>
-      </joint>
-    </xacro:if>
-    <xacro:unless value="${has_podest}">
+  <xacro:include filename="$(find erl_schunk_pg70)/urdf/common.xacro" />
+  <xacro:include filename="$(find erl_schunk_pg70)/urdf/pg70/pg70.gazebo.xacro" />
+  <xacro:include filename="$(find erl_schunk_pg70)/urdf/pg70/pg70.transmission.xacro" />
+  <xacro:macro name="schunk_pg70" params="parent name *origin">
       <joint name="${name}_palm_joint" type="fixed">
         <xacro:insert_block name="origin" />
@@ -38,5 +10,4 @@
         <child link="${name}_palm_link" />
       </joint>
-    </xacro:unless>
     <link name="${name}_palm_link">
       <inertial>
@@ -47,10 +18,10 @@
       <visual>
         <geometry>
-          <mesh filename="package://schunk_description/meshes/pg70/pg70.dae" />
+          <mesh filename="package://erl_schunk_pg70/meshes/pg70/pg70.dae" />
         </geometry>
       </visual>
       <collision>
         <geometry>
-          <mesh filename="package://schunk_description/meshes/pg70/pg70.stl" />
+          <mesh filename="package://erl_schunk_pg70/meshes/pg70/pg70.stl" />
         </geometry>
       </collision>
