Commit message: gripper working on gazebo

File: taurob_schunk_lwa4d/urdf/lwa4d_pg70.urdf.xacro (robot description, xacro)
@@ -16,5 +16,5 @@
   <!-- gripper -->
   <xacro:schunk_pg70 name="pg70" parent="arm_ee_link">
-    <origin xyz="0 0 0" rpy="0 0 0" />
+    <origin xyz="0 0 0" rpy="0 0 0" /> <!--slightly above gazebo plane-->
   </xacro:schunk_pg70>
 </robot>

Commit message: broken name fixed

File: taurob_schunk_lwa4d/urdf/lwa4d_pg70.urdf.xacro (robot description, xacro)
@@ -16,5 +16,5 @@
   <!-- gripper -->
   <xacro:schunk_pg70 name="pg70" parent="arm_ee_link">
-    <origin xyz="0 0 0" rpy="0 0 0" /> <!--slightly above gazebo plane-->
+    <origin xyz="0 0 0" rpy="0 0 0" />
   </xacro:schunk_pg70>
 </robot>

File: taurob_schunk_lwa4d/urdf/schunk_lwa4d_standalone.urdf.xacro (robot description, xacro)
@@ -6,15 +6,9 @@
   <!-- schunk lwa4d -->
   <xacro:include filename="$(find taurob_schunk_lwa4d)/urdf/lwa4d/lwa4d.urdf.xacro" />
-  <!-- schunk pg70 -->
-  <xacro:include filename="$(find erl_schunk_pg70)/urdf/pg70/pg70.urdf.xacro" />
-  <!-- Used for fixing robot to Gazebo -->
+ <!-- Used for fixing robot to Gazebo -->
   <link name="world"/>
-   <!-- arm -->
+  <!-- arm -->
   <xacro:schunk_lwa4d name="arm" parent="world" has_podest="true" use_factory_settings="true">
     <origin xyz="0 0 0" rpy="0 0 0" />
   </xacro:schunk_lwa4d>
-  <!-- gripper -->
-  <xacro:schunk_pg70 name="pg70" parent="arm_ee_link">
-    <origin xyz="0 0 0" rpy="0 0 0" />
-  </xacro:schunk_pg70>
 </robot>
