Commit message: several fixies in model and moveit

File: erl_lwa4d/urdf/lwa4d/lwa4d.urdf.xacro (robot description, xacro)
@@ -1,8 +1,25 @@
 <?xml version="1.0"?>
-<robot xmlns:xacro="http://www.ros.org/wiki/xacro">
+<robot xmlns:xacro="http://www.ros.org/wiki/xacro" name="lwa4d">
   <xacro:property name="safety_offset" value="0.02"/>
   <xacro:include filename="$(find erl_lwa4d)/urdf/common.xacro" />
   <xacro:include filename="$(find erl_lwa4d)/urdf/lwa4d/lwa4d.gazebo.xacro"/>
   <xacro:include filename="$(find erl_lwa4d)/urdf/lwa4d/lwa4d.transmission.xacro"/>
+  <!-- use_factory_setings is a xacro parameter to be used to adapt the urdf according to your hardware setup.
+       use_factory_settings:=true if you have not modified the schunk firmware.
+       use_factory_settings:=false if you have modified the schunk firmware to follow DH parameters (you have inverted the PRL+ motors j1-j5)
+       if you are using custom firmware settings, use schunk_lwa4d_custom
+  -->
+  <xacro:macro name="schunk_lwa4d" params="parent name *origin has_podest:=true use_factory_settings:=true">
+    <xacro:if value="${use_factory_settings}">
+      <xacro:schunk_lwa4d_custom parent="${parent}" name="${name}" has_podest="${has_podest}" invert_j1="false" invert_j2="false" invert_j3="false" invert_j4="false" invert_j5="false" invert_j6="false" invert_j7="false">
+        <xacro:insert_block name="origin" />
+      </xacro:schunk_lwa4d_custom>
+    </xacro:if>
+    <xacro:unless value="${use_factory_settings}">
+      <xacro:schunk_lwa4d_custom parent="${parent}" name="${name}" has_podest="${has_podest}" invert_j1="true" invert_j2="true" invert_j3="true" invert_j4="true" invert_j5="true" invert_j6="true" invert_j7="true">
+        <xacro:insert_block name="origin" />
+      </xacro:schunk_lwa4d_custom>
+    </xacro:unless>
+  </xacro:macro>
   <xacro:macro name="axis_config" params="invert">
     <xacro:if value="${invert}">
@@ -11,21 +28,4 @@
     <xacro:unless value="${invert}">
       <axis xyz="0 0 -1" />
-    </xacro:unless>
-  </xacro:macro>
-  <!-- use_factory_setings is a xacro parameter to be used to adapt the urdf according to your hardware setup.
-       use_factory_settings:=true if you have not modified the schunk firmware.
-       use_factory_settings:=false if you have modified the schunk firmware to follow DH parameters (you have inverted the PRL+ motors j1-j5)
-       if you are using custom firmware settings, use schunk_lwa4d_custom
-  -->
-  <xacro:macro name="schunk_lwa4d" params="parent name *origin has_podest use_factory_settings">
-    <xacro:if value="${use_factory_settings}">
-      <xacro:schunk_lwa4d_custom parent="${parent}" name="${name}" has_podest="${has_podest}" invert_j1="false" invert_j2="false" invert_j3="false" invert_j4="false" invert_j5="false" invert_j6="false" invert_j7="false">
-        <xacro:insert_block name="origin" />
-      </xacro:schunk_lwa4d_custom>
-    </xacro:if>
-    <xacro:unless value="${use_factory_settings}">
-      <xacro:schunk_lwa4d_custom parent="${parent}" name="${name}" has_podest="${has_podest}" invert_j1="true" invert_j2="true" invert_j3="true" invert_j4="true" invert_j5="true" invert_j6="true" invert_j7="true">
-        <xacro:insert_block name="origin" />
-      </xacro:schunk_lwa4d_custom>
     </xacro:unless>
   </xacro:macro>

File: erl_lwa4d/urdf/lwa4d_standalone.urdf.xacro (robot description, xacro)
@@ -1,4 +1,3 @@
-<robot xmlns:xacro="http://www.ros.org/wiki/xacro"
-       name="lwa4d" >
+<robot xmlns:xacro="http://www.ros.org/wiki/xacro" name="lwa4d" >
   <!-- common stuff -->
   <xacro:include filename="$(find erl_lwa4d)/urdf/common.xacro" />

Commit message: new package for jogging

File: erl_lwa4d/urdf/lwa4d/lwa4d.urdf.xacro (robot description, xacro)
@@ -1,5 +1,7 @@
 <?xml version="1.0"?>
 <robot xmlns:xacro="http://www.ros.org/wiki/xacro" name="lwa4d">
-  <xacro:property name="safety_offset" value="0.02"/>
+  <xacro:property name="movement_safety_offset" value="0.05"/>
+  <xacro:property name="velocity_safety_offset" value="0.2"/>
+  <xacro:property name="velocityERB_safety_offset" value="0.5"/>
   <xacro:include filename="$(find erl_lwa4d)/urdf/common.xacro" />
   <xacro:include filename="$(find erl_lwa4d)/urdf/lwa4d/lwa4d.gazebo.xacro"/>
@@ -79,5 +81,5 @@
       <child link="${name}_1_link"/>
       <xacro:axis_config invert="${invert_j1}"/>
-      <limit effort="216" velocity="0.43633" lower="${-M_PI+safety_offset}" upper="${M_PI-safety_offset}"/>
+      <limit effort="216" velocity="${0.43633-velocity_safety_offset}" lower="${-M_PI+movement_safety_offset}" upper="${M_PI-movement_safety_offset}"/>
     </joint>
     <link name="${name}_1_link">
@@ -106,5 +108,5 @@
       <child link="${name}_2_link"/>
       <xacro:axis_config invert="${invert_j2}"/>
-      <limit effort="216" velocity="0.43633" lower="${-2.14 + safety_offset}" upper="${2.14 - safety_offset}"/>
+      <limit effort="216" velocity="${0.43633-velocity_safety_offset}" lower="${-2.14 + movement_safety_offset}" upper="${2.14 - movement_safety_offset}"/>
     </joint>
     <link name="${name}_2_link">
@@ -133,5 +135,5 @@
       <child link="${name}_3_link"/>
       <xacro:axis_config invert="${invert_j3}"/>
-      <limit effort="81.5" velocity="0.4189" lower="${-M_PI + safety_offset}" upper="${M_PI - safety_offset}"/>
+      <limit effort="81.5" velocity="${0.4189-velocity_safety_offset}" lower="${-M_PI + movement_safety_offset}" upper="${M_PI - movement_safety_offset}"/>
     </joint>
     <link name="${name}_3_link">
@@ -160,5 +162,5 @@
       <child link="${name}_4_link"/>
       <xacro:axis_config invert="${invert_j4}"/>
-      <limit effort="81.5" velocity="0.4189" lower="${-2.18 + safety_offset}" upper="${2.18 - safety_offset}"/>
+      <limit effort="81.5" velocity="${0.4189-velocity_safety_offset}" lower="${-2.18 + movement_safety_offset}" upper="${2.18 - movement_safety_offset}"/>
     </joint>
     <link name="${name}_4_link">
@@ -187,5 +189,5 @@
       <child link="${name}_5_link"/>
       <xacro:axis_config invert="${invert_j5}"/>
-      <limit effort="20.7" velocity="0.43633" lower="${-M_PI + safety_offset}" upper="${M_PI - safety_offset}"/>
+      <limit effort="20.7" velocity="${0.43633-velocity_safety_offset}" lower="${-M_PI + movement_safety_offset}" upper="${M_PI - movement_safety_offset}"/>
     </joint>
     <link name="${name}_5_link">
@@ -214,5 +216,5 @@
       <child link="${name}_6_link"/>
       <xacro:axis_config invert="${invert_j6}"/>
-      <limit effort="15" velocity="1.2566" lower="${-2.09 + safety_offset}" upper="${2.09 - safety_offset}"/>
+      <limit effort="15" velocity="${1.2566-velocityERB_safety_offset}" lower="${-2.09 + movement_safety_offset}" upper="${2.09 - movement_safety_offset}"/>
     </joint>
     <link name="${name}_6_link">
@@ -241,5 +243,5 @@
       <child link="${name}_7_link"/>
       <xacro:axis_config invert="${invert_j7}"/>
-      <limit effort="15" velocity="1.2566" lower="${-2.96 + safety_offset}" upper="${2.96 - safety_offset}"/>
+      <limit effort="15" velocity="${1.2566-velocityERB_safety_offset}" lower="${-2.96 + movement_safety_offset}" upper="${2.96 - movement_safety_offset}"/>
     </joint>
     <link name="${name}_7_link">
