Commit message: use of second joystick + 2 cams

File: erl_pg70/urdf/pg70/pg70.urdf.xacro (robot description, xacro)
@@ -32,5 +32,5 @@
       <child link="${name}_finger_left_link" />
       <axis xyz="0 1 0" />
-      <limit effort="10" lower="-0.001" upper="0.061" velocity="2.0"/>
+      <limit effort="5" lower="-0.001" upper="0.03" velocity="1.5"/>
     </joint>
     <link name="${name}_finger_left_link">
